Commit message: Add GY-91 IMU support to Isaac Lab

File: assets/q1/urdf/q1.urdf (robot description, URDF)
Before this commit: robot YSXSZ, 12 links, 11 joints
Links:
- link imu_in_torso: geometry visual mesh filename=../meshes/GY_91.STL scale=0.001 0.001 0.001
Joints:
- joint imu_in_torso_joint: origin xyz=0.033 0. 0.015 rpy=0 0 0 -> xyz=0.163 0 0.025 rpy=0 0 -1.5707963
